Commit message: Modification of main class to sonar

File: xacro/gazebo_magnet_test.xacro (robot description, xacro)
@@ -1,11 +1,16 @@
 <?xml version="1.0"?>
 <robot xmlns:xacro="http://www.ros.org/wiki/xacro">
-<gazebo>
+<gazebo reference="car_sonar/base_link">
+<sensor name='my_contact' type='camera'>
     <plugin name="SonarVisual" filename="libSonarVisual.so" >
-        <horizontal_fov>${hfov}</horizontal_fov>
+        <horizontal_fov>${pi}</horizontal_fov>
         <image>
             <width>100</width>
             <height>100</height>
-            <format>R8G8B8</format>
+            <format>R32G32B32</format>
+<<<<<<< HEAD
+>>>>>>> 3db1d56... Modification of main class to sonar
+=======
+>>>>>>> 7c8862b... 2
         </image>
         <clip>
@@ -19,4 +24,9 @@
         </noise>
     </plugin>
+</sensor>
+<<<<<<< HEAD
+>>>>>>> 3db1d56... Modification of main class to sonar
+=======
+>>>>>>> 7c8862b... 2
 </gazebo>
 </robot>

File: xacro/sensors_magnet_test.xacro (robot description, xacro)
@@ -2,5 +2,5 @@
 <robot xmlns:xacro="http://www.ros.org/wiki/xacro">
 <xacro:default_camera namespace="${namespace}" parent_link="${namespace}/base_link" suffix="down">
-    <origin xyz="1 1 1 " rpy="0 0 0"/>
+    <origin xyz="0 0 1 " rpy="0 ${pi/2} 0"/>
   </xacro:default_camera>
 </robot>
