Commit message: Files Organization of Shader implementation

File: xacro/base_magnet_test.xacro (robot description, xacro)
@@ -45,4 +45,34 @@
       <selfCollide>false</selfCollide>
     </gazebo>
+    <link name="${namespace}/test_link">
+      <!--
+          Be careful to setup the coefficients for the inertial tensor,
+          otherwise your model will become unstable on Gazebo
+        -->
+      <inertial>
+        <mass value="0.01"/>
+        <origin xyz="0 0 0" rpy="0 0 0"/>
+        <inertia ixx="0.01" ixy="0.001" ixz="0.001" iyy="0.01" iyz="0.001" izz="0.01"/>
+      </inertial>
+      <!-- <visual>
+        <origin xyz="0 0 0" rpy="0 0 0"/>
+        <geometry>
+          <box size="0.4 0.8 0.1"/>
+        </geometry>
+      </visual> -->
+      <collision>
+        <origin xyz="0 0 0" rpy="0 0 0"/>
+        <geometry>
+          <box size="0.001 0.001 0.001"/>
+        </geometry>
+      </collision>
+    </link>
+    <joint name="${namespace}/test_joint" type="revolute">
+      <origin xyz="0 0 3" rpy="0 ${pi/2} ${pi/2}"/>
+      <parent link="${namespace}/base_link" />
+      <child link="${namespace}/test_link" />
+      <limit upper="0" lower="0" effort="0" velocity="0" />
+      <axis xyz="1 0 0"/>
+    </joint>
     <!-- Set up hydrodynamic plugin given as input parameter -->
     <xacro:insert_block name="gazebo"/>

File: xacro/gazebo_magnet_test.xacro (robot description, xacro)
@@ -1,11 +1,15 @@
 <?xml version="1.0"?>
 <robot xmlns:xacro="http://www.ros.org/wiki/xacro">
-<gazebo reference="car_sonar/base_link">
+<gazebo reference="car_sonar/test_link">
 <sensor name='my_contact' type='camera'>
-    <plugin name="SonarVisual" filename="libSonarVisual.so" >
-        <horizontal_fov>${pi}</horizontal_fov>
+    <plugin name="SonarVisual" filename="libfl_sonar_ros.so" >
+        <link_reference>car_sonar/test_link</link_reference>
+        <horizontal_fov>${pi/2}</horizontal_fov>
+        <vfov>${pi/4}</vfov>
+        <bin_count>720</bin_count>
+        <beam_count>720</beam_count>
         <image>
-            <width>100</width>
-            <height>100</height>
+            <width>720</width>
+            <height>720</height>
             <format>R32G32B32</format>
 <<<<<<< HEAD
@@ -16,5 +20,5 @@
         <clip>
             <near>0.1</near>
-            <far>3000</far>
+            <far>5</far>
         </clip>
         <noise>
