Commit message: Tests inclusion 	- Final formating 	- Gazebo tests for shader and image manipulation

File: xacro/base_car_sonar.xacro (robot description, xacro)
@@ -2,5 +2,5 @@
 <robot xmlns:xacro="http://www.ros.org/wiki/xacro">
   <!-- Loading concept -->
-  <xacro:property name="concept" value="magnet_test"/>
+  <xacro:property name="concept" value="car_sonar"/>
   <!-- Loading vehicle's specific macros -->
   <xacro:include filename="$(find  gazebo_ros_sonar_plugin)/xacro/snippets_${concept}.xacro"/>
@@ -78,7 +78,7 @@
     <xacro:insert_block name="gazebo"/>
     <!-- Include the thruster modules -->
-    <xacro:include filename="$(find gazebo_ros_sonar_plugin)/xacro/actuators_magnet_test.xacro"/>
+    <xacro:include filename="$(find gazebo_ros_sonar_plugin)/xacro/actuators_car_sonar.xacro"/>
     <!-- Include the sensor modules -->
-    <xacro:include filename="$(find gazebo_ros_sonar_plugin)/xacro/sensors_magnet_test.xacro"/>
+    <xacro:include filename="$(find gazebo_ros_sonar_plugin)/xacro/sensors_car_sonar.xacro"/>
   </xacro:macro>
 </robot>

File: xacro/default_car_sonar.xacro (robot description, xacro)
@@ -2,6 +2,6 @@
 <robot xmlns:xacro="http://www.ros.org/wiki/xacro" name="mccr">
   <xacro:arg name="debug" default="0"/>
-  <xacro:arg name="namespace" default="mccr"/>
-  <xacro:arg name="concept" default="magnet_test"/>
+  <xacro:arg name="namespace" default="car_sonar"/>
+  <xacro:arg name="concept" default="car_sonar"/>
   <!-- -->
   <!-- Include the ROV macro file -->

File: xacro/gazebo_car_sonar.xacro (robot description, xacro)
@@ -2,6 +2,7 @@
 <robot xmlns:xacro="http://www.ros.org/wiki/xacro">
 <gazebo reference="car_sonar/test_link">
-<sensor name='my_contact' type='camera'>
+<sensor name='FLSonar' type='camera'>
     <plugin name="SonarVisual" filename="libfl_sonar_ros.so" >
+        <topic>car_sonar/FLSonar</topic>
         <link_reference>car_sonar/test_link</link_reference>
         <horizontal_fov>${pi/2}</horizontal_fov>
